Commit message: Fixed nonvisible robot model, need to add jsp

File: autogiro/description/robot.urdf.xacro (robot description, xacro)
@@ -2,5 +2,5 @@
 <robot xmlns:xacro="http://www.ros.org/wiki/xacro"  name="robot">
     <xacro:arg name="use_ros2_control" default="true"/>
-    <xacro:arg name="sim_mode" default="false"/>
+    <xacro:arg name="sim_mode" default="true"/>
     <xacro:include filename="robot_core.xacro" />
     <xacro:if value="$(arg use_ros2_control)">

File: autogiro/description/robot_core.xacro (robot description, xacro)
@@ -15,5 +15,5 @@
     <xacro:property name="caster_mass" value="1.1"/>
     <xacro:property name="caster_thickness" value=".058"/>
-    <xacro:property name="caster_offset_x" value="1.68"/>
+    <xacro:property name="caster_offset_x" value="0.68"/>
     <xacro:property name="caster_offset_z" value="${wheel_offset_z - wheel_radius + caster_radius}"/>
     <xacro:property name="caster_offset_y" value="0.27"/>
