Commit message: Sync update package and cmake for Ubuntu

File: autogiro/description/robot_core.xacro (robot description, xacro)
@@ -56,5 +56,5 @@
                 <box size="${chassis_length} ${chassis_width} ${chassis_height}"/>
             </geometry>
-            <material name="Orange"/>
+            <material name="orange"/>
         </visual>
         <collision>

File: autogiro/description/ros2_control.xacro (robot description, xacro)
@@ -58,5 +58,6 @@
     </xacro:if>
     <gazebo>
-        <plugin name="gazebo_ros2_control" filename="libgazebo_ros2_control.dylib"> <!-- changed from .so to .dylib -->
+        <!-- <plugin name="gazebo_ros2_control" filename="libgazebo_ros2_control.dylib"> changed from .so to .dylib -->
+            <plugin name="gazebo_ros2_control" filename="libgazebo_ros2_control.so"> <!-- Reverted to play around with loading logic-->
             <parameters>$(find autogiro)/config/my_controllers.yaml</parameters>
             <parameters>$(find autogiro)/config/gaz_ros2_ctl_use_sim.yaml</parameters>
