Commit message: bot visible in gazebo, falls through floor though

File: autogiro/description/inertial_macros.xacro (robot description, xacro)
@@ -28,5 +28,5 @@
             <inertia ixx="${(1/12) * mass * (3*radius*radius + length*length)}" ixy="0.0" ixz="0.0"
                     iyy="${(1/12) * mass * (3*radius*radius + length*length)}" iyz="0.0"
-                    izz="0.135" /> <!-- changed from formula to 0.135 to match motor inertia, reference articubot for old-->
+                    izz="${(mass/2.0) * (radius*radius)}" />  articubot for old-->
         </inertial>
     </xacro:macro>

File: autogiro/description/robot_core.xacro (robot description, xacro)
@@ -7,5 +7,5 @@
     <xacro:property name="chassis_mass" value="68.039"/>
     <xacro:property name="wheel_radius" value=".161"/>
-    <xacro:property name="wheel_thickness" value="0.055"/>
+    <xacro:property name="wheel_thickness" value="0.055"/> <!-- Changed to fix error code 18 from phys engine (was 0.055) -->
     <xacro:property name="wheel_mass" value=".725"/>
     <xacro:property name="wheel_offset_x" value="0.0"/>
