Commit message: Lidar on chassis, working on gazebo startup

File: autogiro/description/lidar.xacro (robot description, xacro)
@@ -4,10 +4,10 @@
         <parent link="chassis"/>
         <child link="laser_frame"/>
-        <origin xyz="0.122 0 0.212" rpy="0 0 0"/>
+        <origin xyz="0.1 0 1.8 " rpy="0 0 0"/> <!-- 1.8m is the height of the lidar from the ground -->
     </joint>
     <link name="laser_frame">
         <visual>
             <geometry>
-                <cylinder radius="0.05" length="0.04"/>
+                <cylinder radius="0.0325" length="0.06"/>
             </geometry>
             <material name="black"/>
@@ -16,5 +16,5 @@
             <origin xyz="0 0 -0.05"/>
             <geometry>
-                <cylinder radius="0.01" length="0.1"/>
+                <cylinder radius="0.0325" length="0.06"/>
             </geometry>
             <material name="black"/>
@@ -22,8 +22,8 @@
         <collision>
             <geometry>
-                <cylinder radius="0.05" length="0.04"/>
+                <cylinder radius="0.0325" length="0.06"/>
             </geometry>
         </collision>
-        <xacro:inertial_cylinder mass="0.1" length="0.04" radius="0.05">
+        <xacro:inertial_cylinder mass="0.1" length="0.06" radius="0.0325">
             <origin xyz="0 0 0" rpy="0 0 0"/>
         </xacro:inertial_cylinder>
@@ -31,22 +31,22 @@
     <gazebo reference="laser_frame">
         <material>Gazebo/Black</material>
-        <sensor name="laser" type="ray">
+        <sensor name="laser" type="gpu_lidar">
             <pose> 0 0 0 0 0 0 </pose>
             <visualize>false</visualize>
-            <update_rate>10</update_rate>
-            <ray>
+            <update_rate>10</update_rate> <!-- 10 Hz -->
+            <gpu_lidar>
                 <scan>
                     <horizontal>
                         <samples>360</samples>
-                        <min_angle>-3.14</min_angle>
-                        <max_angle>3.14</max_angle>
+                        <min_angle>-0.0976</min_angle> <!-- -52 degrees -->
+                        <max_angle>0.1222</max_angle> <!-- 7 degrees -->
                     </horizontal>
                 </scan>
                 <range>
-                    <min>0.3</min>
-                    <max>12</max>
+                    <min>0.1</min>
+                    <max>20</max>
                 </range>
-            </ray>
-            <plugin name="laser_controller" filename="libgazebo_ros_ray_sensor.so">
+            </gpu_lidar>
+            <!-- <plugin name="laser_controller" filename="libgazebo_ros_gpu_laser.so">
                 <ros>
                     <argument>~/out:=scan</argument>
@@ -54,5 +54,5 @@
                 <output_type>sensor_msgs/LaserScan</output_type>
                 <frame_name>laser_frame</frame_name>
-            </plugin>
+            </plugin> -->
         </sensor>
     </gazebo>

File: autogiro/description/robot.urdf.xacro (robot description, xacro)
@@ -4,4 +4,5 @@
     <xacro:arg name="sim_mode" default="true"/>
     <xacro:include filename="robot_core.xacro" />
+    <xacro:include filename="lidar.xacro" />
     <xacro:if value="$(arg use_ros2_control)">
         <xacro:include filename="ros2_control.xacro" />
@@ -10,4 +11,3 @@
         <xacro:include filename="gazebo_control.xacro" />
     </xacro:unless>
-    <xacro:include filename="lidar.xacro" />
 </robot>

File: autogiro/description/robot_core.xacro (robot description, xacro)
@@ -56,5 +56,5 @@
                 <box size="${chassis_length} ${chassis_width} ${chassis_height}"/>
             </geometry>
-            <material name="orange"/>
+            <material name="Orange"/>
         </visual>
         <collision>
@@ -64,5 +64,5 @@
             </geometry>
         </collision>
-        <xacro:inertial_box mass="0.5" x="${chassis_length}" y="${chassis_width}" z="${chassis_height}">
+        <xacro:inertial_box mass="${chassis_mass}" x="${chassis_length}" y="${chassis_width}" z="${chassis_height}">
             <origin xyz="${chassis_length/2} 0 ${chassis_height/2}" rpy="0 0 0"/>
         </xacro:inertial_box>

File: autogiro/description/ros2_control.xacro (robot description, xacro)
@@ -55,5 +55,5 @@
     </xacro:if>
     <gazebo>
-        <plugin name="gazebo_ros2_control" filename="libgazebo_ros2_control.so">
+        <plugin name="gazebo_ros2_control" filename="libgazebo_ros2_control.dylib"> <!-- changed from .so to .dylib -->
             <parameters>$(find autogiro)/config/my_controllers.yaml</parameters>
             <parameters>$(find autogiro)/config/gaz_ros2_ctl_use_sim.yaml</parameters>

Commit message: Lidar publishing, check in Rviz2

File: autogiro/description/lidar.xacro (robot description, xacro)
@@ -4,5 +4,5 @@
         <parent link="chassis"/>
         <child link="laser_frame"/>
-        <origin xyz="0.1 0 1.8 " rpy="0 0 0"/> <!-- 1.8m is the height of the lidar from the ground -->
+        <origin xyz="0.1 0 1.8 " rpy="${pi} 0 0"/> <!-- 1.8m is the height of the lidar from the ground -->
     </joint>
     <link name="laser_frame">
@@ -33,13 +33,19 @@
         <sensor name="laser" type="gpu_lidar">
             <pose> 0 0 0 0 0 0 </pose>
-            <visualize>false</visualize>
-            <update_rate>10</update_rate> <!-- 10 Hz -->
+            <visualize>true</visualize>
+            <update_rate>10</update_rate> <topic>scan</topic> <!-- 10 Hz -->
+            <gz_frame_id>laser_frame</gz_frame_id>
             <gpu_lidar>
                 <scan>
                     <horizontal>
-                        <samples>360</samples>
-                        <min_angle>-0.0976</min_angle> <!-- -52 degrees -->
-                        <max_angle>0.1222</max_angle> <!-- 7 degrees -->
+                    	<samples>360</samples>
+                        <resolution>1</resolution>
+                        <min_angle>-3.14159</min_angle>
+                        <max_angle>3.14159</max_angle>
                     </horizontal>
+                    <vertical>
+                        <samples>16</samples> <resolution>1</resolution>
+                        <min_angle>-0.9076</min_angle> <max_angle>0.1222</max_angle>
+                    </vertical>
                 </scan>
                 <range>

Commit message: robot model fixed, lidar orientation corrected. Need to work on sync, no /scan feed

File: autogiro/description/lidar.xacro (robot description, xacro)
@@ -2,7 +2,7 @@
 <robot xmlns:xacro="http://www.ros.org/wiki/xacro" >
     <joint name="laser_joint" type="fixed">
-        <parent link="chassis"/>
+        <parent link="mast"/>
         <child link="laser_frame"/>
-        <origin xyz="0.1 0 1.8 " rpy="${pi} 0 0"/> <!-- 1.8m is the height of the lidar from the ground -->
+        <origin xyz="0.1 0 0.73" rpy="${pi} 0 0"/>
     </joint>
     <link name="laser_frame">
@@ -48,6 +48,6 @@
                         <samples>16</samples>
                         <resolution>1</resolution>
-                        <min_angle>-0.9076</min_angle>
-                        <max_angle>0.1222</max_angle>
+                        <min_angle>-0.1222</min_angle>
+                        <max_angle>0.9076</max_angle>
                     </vertical>
                 </scan>

File: autogiro/description/robot_core.xacro (robot description, xacro)
@@ -44,30 +44,79 @@
     <link name="base_footprint">
     </link>
-    <!-- CHASSIS LINK -->
-    <joint name="chassis_joint" type="fixed">
-        <parent link="base_link"/>
-        <child link="chassis"/>
+    <!-- CHASSIS BASE LINK -->
+    <joint name="chassis_base_joint" type="fixed">
+        <parent link="base_link"/>
+        <child link="chassis_base"/>
         <origin xyz="${-wheel_offset_x} 0 ${-wheel_offset_z}"/>
     </joint>
-    <link name="chassis">
-        <visual>
-            <origin xyz="${chassis_length/2} 0 ${chassis_height/2}"/>
-            <geometry>
-                <box size="${chassis_length} ${chassis_width} ${chassis_height}"/>
+    <link name="chassis_base">
+        <visual>
+            <origin xyz="${chassis_length/2} 0 ${chassis_height/2 - 0.3}"/>
+            <geometry>
+                <box size="${chassis_length} ${chassis_width} ${chassis_height-0.7}"/>
             </geometry>
             <material name="orange"/>
         </visual>
         <collision>
-            <origin xyz="${chassis_length/2} 0 ${chassis_height/2}"/>
-            <geometry>
-                <box size="${chassis_length} ${chassis_width} ${chassis_height}"/>
+            <origin xyz="${chassis_length/2} 0 0.535"/>
+            <geometry>
+                <box size="${chassis_length} ${chassis_width} ${chassis_height-0.7}"/>
             </geometry>
         </collision>
         <xacro:inertial_box mass="${chassis_mass}" x="${chassis_length}" y="${chassis_width}" z="${chassis_height}">
-            <origin xyz="${chassis_length/2} 0 ${chassis_height/2}" rpy="0 0 0"/>
+            <origin xyz="${chassis_length/2} 0 0.535" rpy="0 0 0"/>
         </xacro:inertial_box>
     </link>
-    <gazebo reference="chassis">
+    <gazebo reference="chassis_base">
         <material>Gazebo/Orange</material>
+    </gazebo>
+    <!-- LIDAR MAST LINK -->
+    <joint name="mast_joint" type="fixed">
+        <parent link="chassis_base" />
+        <child link="mast" />
+        <origin xyz="0 0 1.07" rpy="0 0 0" />
+    </joint>
+    <link name="mast">
+        <visual>
+            <origin xyz="0 0 0.365" rpy="0 0 0" /> <geometry>
+                <box size="0.05 0.05 0.73" /> </geometry>
+            <material name="white" />
+        </visual>
+        <collision>
+            <origin xyz="0 0 0.365" rpy="0 0 0" />
+            <geometry>
+                <box size="0.05 0.05 0.73" />
+            </geometry>
+        </collision>
+        <xacro:inertial_box mass="5.0" x=".05" y=".05" z="0.365">
+            <origin xyz="${chassis_length/2} 0 0.535" rpy="0 0 0"/>
+        </xacro:inertial_box>
+    </link>
+    <gazebo reference="mast">
+        <material>Gazebo/White</material>
+    </gazebo>
+    <!-- SEAT LINK -->
+    <joint name="seat_joint" type="fixed">
+        <parent link="chassis_base" />
+        <child link="seat" />
+        <origin xyz="0.465 0 1.07" rpy="0 0 0" /> </joint>
+    <link name="seat">
+        <visual>
+            <origin xyz="0 0 -0.05" rpy="0 0 0" /> <geometry>
+                <box size="0.5 0.5 0.5" /> </geometry>
+            <material name="blue" />
+        </visual>
+        <collision>
+            <origin xyz="0 0 0.25" rpy="0 0 0" />
+            <geometry>
+                <box size="0.5 0.5 0.5" />
+            </geometry>
+        </collision>
+        <xacro:inertial_box mass="10.0" x="0" y="0" z="0.25">
+            <origin xyz="0 0 0.25" rpy="0 0 0"/>
+        </xacro:inertial_box>
+    </link>
+    <gazebo reference="seat">
+        <material>Gazebo/Blue</material>
     </gazebo>
     <!-- LEFT WHEEL LINK -->
